Commit message: .

File: rosbee_ros/rosbee_description/urdf/components/bottom_plate.urdf.xacro (robot description, xacro)
@@ -1,4 +1,5 @@
 <?xml version="1.0"?>
 <robot xmlns:xacro="http://www.ros.org/wiki/xacro" name="rosbee">
+  <property name="M_PI" value="3.14159"/>
   <!-- bottom_plate properties -->
   <property name="bottom_diameter" value="0.390" />
@@ -11,5 +12,5 @@
         <mesh filename="package://rosbee_description/meshes/500068B_rosbee_base_plate_350.stl" scale="0.001 0.001 0.001"/>
       </geometry>
-      <origin rpy="0 0 0" xyz="0 0 ${bottom_plate_offset_z}"/>
+      <origin rpy="0 0 ${M_PI}" xyz="0 0 ${bottom_plate_offset_z}"/>
       <material name="black">
         <color rgba="0.1 0.1 0.1 1"/>
