Commit message: config changes

File: rosbee_ros/rosbee_description/robots/rosbee.urdf.xacro (robot description, xacro)
@@ -54,6 +54,12 @@
                           offset_z="-0.0050"/>
   <!--  kinect sensor -->
-  <xacro:sensor_kinect parent="top_plate_link">
+  <!--<xacro:sensor_kinect parent="top_plate_link">
     <origin xyz="-0.100 0.0000 0.126" rpy="0 0 0"/>
-  </xacro:sensor_kinect>
+  </xacro:sensor_kinect>-->
+  <joint name="depth_sensor_joint" type="fixed">
+      <origin xyz="-0.100 0.000 0.126" rpy="0 0 0"/>
+      <child link="camera_link"/>
+      <parent link="top_plate_link"/>
+  </joint>
+  <link name="camera_link"/>
 </robot>
